File: kicad/mdb-slave-esp32s3.kicad_sch (KiCad schematic)
At the start: 35 parts, among them J1 MDB_Connector, J2 USB_C_Receptacle_USB2.0_16P, J3 Conn_02x11_Odd_Even, SW1 SW_Push, U1 TLP785, U2 KA78M05_TO252, U3 ESP32-S3FH4R2, U4 TLP785, Y1 Crystal_GND24

Commit message: Update KiCad project and add schematic
Parts:
- added C2: 0.1uF, Capacitor_SMD:C_0603_1608Metric, symbol Device:C
- added C3: 220pF, Capacitor_SMD:C_0603_1608Metric, symbol Device:C
- added D1: 1N4148WT, Diode_SMD:D_SOD-523, symbol Diode:1N4148WT
- added D4, D6: ESD5Z12V, Diode_SMD:D_SOD-523, symbol Diode:ESD5Zxx
- added U5: 74LVC1G14, symbol 74xGxx:74LVC1G14
- R1: value 10K -> 4.7K
- R2: value 470ohm -> 3.9K
Connections:
- net +3V3: now also C2.2, U5.5 (VCC)
- net GND: now also C2.1, C3.2, U5.3 (GND)
- net io4: now also U5.4; no longer R1.1, U4.4
- net mdb_communications_common: now also D1.2 (A), D4.2 (A), D6.2 (A)
- net mdb_master_receive: now also D6.1 (K)
- net mdb_master_transmit: now also D4.1 (K)
- net at R2.2, U4.1: now also D1.1 (K)
- new net: C3.1, R1.1, U4.4, U5.2
Other:
- moved on the sheet: C10, C7, C9, J1, R1, R2, R5, U1, U2, U4
